File: hardware/pcb/Landing-Light/Landing-Light.kicad_sch (KiCad schematic)
At the start: 54 parts, among them J1 Conn_01x04, J2 2012670005, J3 Conn_01x04, Q1 PMOS, Q2 NMOS, SW2 SW_SP3T, SW3 SW_SPDT, U1 BQ25172DSGR, U3 TPS61200DRC

Commit message: Changing to new layout
Parts:
- removed TP1: +BATT, TestPoint:TestPoint_Pad_D1.0mm, symbol Connector:TestPoint
- D2: now not fitted
- D3, D4: now in the parts list
- J3: now not fitted; now left out of the parts list
Connections:
- net VBUS: no longer C8.1, C9.2, FB1.1, J1.4 (Pin_4), J2.A4 (VBUS1), J2.A9 (VBUS2), J2.B4 (VBUS3), J2.B9 (VBUS4), J3.4 (Pin_4)
- new net VSS: C8.1, C9.2, FB1.1, J1.4 (Pin_4), J2.A4 (VBUS1), J2.A9 (VBUS2), J2.B4 (VBUS3), J2.B9 (VBUS4), J3.4 (Pin_4)
Changed lines of the file:
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@@
 		)
 	)
-	(label "VBUS"
-		(at 105.41 46.99 0)
-		(fields_autoplaced yes)
-		(effects
-			(font
-				(size 1.27 1.27)
-			)
-			(justify left bottom)
-		)
-	)
 	(label "CC1"
 		(at 54.61 57.15 0)
@@
 		)
 	)
-	(label "VBUS"
-		(at 35.56 137.16 0)
-		(fields_autoplaced yes)
-		(effects
-			(font
-				(size 1.27 1.27)
-			)
-			(justify left bottom)
-		)
-	)
 	(label "CC2"
 		(at 173.99 78.74 0)
@@
 		)
 	)
-	(label "VBUS"
-		(at 35.56 113.03 0)
-		(fields_autoplaced yes)
-		(effects
-			(font
-				(size 1.27 1.27)
-			)
-			(justify left bottom)
-		)
-	)
 	(global_label "DATA1"
 		(shape input)
@@
 		(exclude_from_sim no)
 		(in_bom no)
-		(on_board yes)
-		(dnp no)
+		(on_board no)
+		(dnp yes)
 		(fields_autoplaced yes)
 		(property "Reference" "D2"
@@
 	)
 	(symbol
+		(lib_id "power:VSS")
+		(at 35.56 113.03 0)
+		(unit 1)
+		(exclude_from_sim no)
+		(in_bom yes)
+		(on_board yes)
+		(dnp no)
+		(fields_autoplaced yes)
+		(property "Reference" "#PWR09"
+			(at 35.56 116.84 0)
+			(effects
+				(font
+					(size 1.27 1.27)
+				)
+				(hide yes)
+			)
+		)
+		(property "Value" "VSS"
+			(at 35.56 107.95 0)
+			(effects
+				(font
+					(size 1.27 1.27)
+				)
+			)
+		)
+		(property "Footprint" ""
+			(at 35.56 113.03 0)
+			(effects
+				(font
+					(size 1.27 1.27)
+				)
+				(hide yes)
+			)
+		)
+		(property "Datasheet" ""
+			(at 35.56 113.03 0)
+			(effects
+				(font
+					(size 1.27 1.27)
+				)
+				(hide yes)
+			)
+		)
+		(property "Description" "Power symbol creates a global label with name \"VSS\""
+			(at 35.56 113.03 0)
+			(effects
+				(font
+					(size 1.27 1.27)
+				)
+				(hide yes)
+			)
+		)
+		(pin "1"
+		)
+		(instances
+			(project "Landing-Light"
+				(path "/f89d3217-1b1a-43a4-8c74-9ff6f0eaa6ee"
+					(reference "#PWR09")
+					(unit 1)
+				)
+			)
+		)
+	)
+	(symbol
 		(lib_id "power:GND")
 		(at 227.33 135.89 0)
@@
 	)
 	(symbol
-		(lib_id "Connector:TestPoint")
-		(at 118.11 217.17 0)
-		(unit 1)
-		(exclude_from_sim no)
-		(in_bom yes)
-		(on_board yes)
-		(dnp no)
-		(fields_autoplaced yes)
-		(property "Reference" "TP1"
-			(at 120.65 212.5979 0)
-			(effects
-				(font
-					(size 1.27 1.27)
-				)
-				(justify left)
-			)
-		)
-		(property "Value" "+BATT"
-			(at 120.65 215.1379 0)
-			(effects
-				(font
-					(size 1.27 1.27)
-				)
-				(justify left)
-			)
-		)
-		(property "Footprint" "TestPoint:TestPoint_Pad_D1.0mm"
-			(at 123.19 217.17 0)
-			(effects
-				(font
-					(size 1.27 1.27)
-				)
-				(hide yes)
-			)
-		)
-		(property "Datasheet" "~"
-			(at 123.19 217.17 0)
-			(effects
-				(font
-					(size 1.27 1.27)
-				)
-				(hide yes)
-			)
-		)
-		(property "Description" "test point"
-			(at 118.11 217.17 0)
-			(effects
-				(font
-					(size 1.27 1.27)
-				)
-				(hide yes)
-			)
-		)
-		(pin "1"
-		)
-		(instances
-			(project "Landing-Light"
-				(path "/f89d3217-1b1a-43a4-8c74-9ff6f0eaa6ee"
-					(reference "TP1")
-					(unit 1)
-				)
-			)
-		)
-	)
-	(symbol
 		(lib_id "Jumper:Jumper_2_Open")
 		(at 298.45 165.1 90)
@@
 	)
 	(symbol
+		(lib_id "power:VSS")
+		(at 110.49 46.99 0)
+		(unit 1)
+		(exclude_from_sim no)
+		(in_bom yes)
+		(on_board yes)
+		(dnp no)
+		(fields_autoplaced yes)
+		(property "Reference" "#PWR08"
+			(at 110.49 50.8 0)
+			(effects
+				(font
+					(size 1.27 1.27)
+				)
+				(hide yes)
+			)
+		)
+		(property "Value" "VSS"
+			(at 110.49 41.91 0)
+			(effects
+				(font
+					(size 1.27 1.27)
+				)
+			)
+		)
+		(property "Footprint" ""
+			(at 110.49 46.99 0)
+			(effects
+				(font
+					(size 1.27 1.27)
+				)
+				(hide yes)
+			)
+		)
+		(property "Datasheet" ""
+			(at 110.49 46.99 0)
+			(effects
+				(font
+					(size 1.27 1.27)
+				)
+				(hide yes)
+			)
+		)
+		(property "Description" "Power symbol creates a global label with name \"VSS\""
+			(at 110.49 46.99 0)
+			(effects
+				(font
+					(size 1.27 1.27)
+				)
+				(hide yes)
+			)
+		)
+		(pin "1"
+		)
+		(instances
+			(project "Landing-Light"
+				(path "/f89d3217-1b1a-43a4-8c74-9ff6f0eaa6ee"
+					(reference "#PWR08")
+					(unit 1)
+				)
+			)
+		)
+	)
+	(symbol
 		(lib_id "Device:R_US")
 		(at 40.64 233.68 0)
@@
 	)
 	(symbol
+		(lib_id "power:VSS")
+		(at 35.56 137.16 0)
+		(unit 1)
+		(exclude_from_sim no)
+		(in_bom yes)
+		(on_board yes)
+		(dnp no)
+		(fields_autoplaced yes)
+		(property "Reference" "#PWR015"
+			(at 35.56 140.97 0)
+			(effects
+				(font
+					(size 1.27 1.27)
+				)
+				(hide yes)
+			)
+		)
+		(property "Value" "VSS"
+			(at 35.56 132.08 0)
+			(effects
+				(font
+					(size 1.27 1.27)
+				)
+			)
+		)
+		(property "Footprint" ""
+			(at 35.56 137.16 0)
+			(effects
+				(font
+					(size 1.27 1.27)
+				)
+				(hide yes)
+			)
+		)
+		(property "Datasheet" ""
+			(at 35.56 137.16 0)
+			(effects
+				(font
+					(size 1.27 1.27)
+				)
+				(hide yes)
+			)
+		)
+		(property "Description" "Power symbol creates a global label with name \"VSS\""
+			(at 35.56 137.16 0)
+			(effects
+				(font
+					(size 1.27 1.27)
+				)
+				(hide yes)
+			)
+		)
+		(pin "1"
+		)
+		(instances
+			(project "Landing-Light"
+				(path "/f89d3217-1b1a-43a4-8c74-9ff6f0eaa6ee"
+					(reference "#PWR015")
+					(unit 1)
+				)
+			)
+		)
+	)
+	(symbol
 		(lib_id "Device:R_US")
 		(at 31.75 241.3 0)
@@
 		(unit 1)
 		(exclude_from_sim no)
-		(in_bom yes)
-		(on_board yes)
-		(dnp no)
+		(in_bom no)
+		(on_board no)
+		(dnp yes)
 		(fields_autoplaced yes)
 		(property "Reference" "J3"
@@
 		(unit 1)
 		(exclude_from_sim no)
-		(in_bom no)
+		(in_bom yes)
 		(on_board yes)
 		(dnp no)
@@
 		(unit 1)
 		(exclude_from_sim no)
-		(in_bom no)
+		(in_bom yes)
 		(on_board yes)
 		(dnp no)

Commit message: Reinstating USB-C
Parts:
- D2: now fitted; now in the parts list
Changed lines of the file:
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@@
 		(unit 1)
 		(exclude_from_sim no)
-		(in_bom no)
-		(on_board no)
-		(dnp yes)
+		(in_bom yes)
+		(on_board yes)
+		(dnp no)
 		(fields_autoplaced yes)
 		(property "Reference" "D2"

Commit message: Tidying up layout
Connections:
- net -BATT: now also R14.2
- net VBUS: now also Q1.1 (G), R14.1; no longer R14.2
Other:
- moved on the sheet: D2, D4
Changed lines of the file:
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@@
 	)
 	(junction
+		(at 176.53 238.76)
+		(diameter 0)
+		(color 0 0 0 0)
+	)
+	(junction
 		(at 204.47 113.03)
 		(diameter 0)
@@
 	)
 	(junction
-		(at 176.53 238.76)
-		(diameter 0)
-		(color 0 0 0 0)
-	)
-	(junction
 		(at 224.79 133.35)
 		(diameter 0)
@@
 	)
 	(junction
+		(at 154.94 227.33)
+		(diameter 0)
+		(color 0 0 0 0)
+	)
+	(junction
 		(at 96.52 52.07)
 		(diameter 0)
@@
 	)
 	(no_connect
-		(at 121.92 78.74)
+		(at 121.92 71.12)
 	)
 	(no_connect
@@
 	(wire
 		(pts
-			(xy 154.94 224.79) (xy 154.94 228.6)
+			(xy 154.94 224.79) (xy 154.94 227.33)
 		)
 		(stroke
@@
 	(wire
 		(pts
-			(xy 176.53 238.76) (xy 154.94 238.76)
-		)
-		(stroke
-			(width 0)
-			(type default)
-		)
-	)
-	(wire
-		(pts
 			(xy 93.98 49.53) (xy 96.52 49.53)
 		)
@@
 	(wire
 		(pts
-			(xy 165.1 82.55) (xy 165.1 86.36)
+			(xy 165.1 74.93) (xy 165.1 78.74)
 		)
 		(stroke
@@
 	(wire
 		(pts
-			(xy 130.81 82.55) (xy 130.81 86.36)
+			(xy 130.81 74.93) (xy 130.81 78.74)
 		)
 		(stroke
@@
 	(wire
 		(pts
+			(xy 154.94 227.33) (xy 154.94 228.6)
+		)
+		(stroke
+			(width 0)
+			(type default)
+		)
+	)
+	(wire
+		(pts
 			(xy 130.81 46.99) (xy 138.43 46.99)
 		)
@@
 	(wire
 		(pts
-			(xy 154.94 238.76) (xy 154.94 236.22)
-		)
-		(stroke
-			(width 0)
-			(type default)
-		)
-	)
-	(wire
-		(pts
 			(xy 31.75 222.25) (xy 31.75 237.49)
 		)
@@
 	(wire
 		(pts
+			(xy 154.94 227.33) (xy 170.18 227.33)
+		)
+		(stroke
+			(width 0)
+			(type default)
+		)
+	)
+	(wire
+		(pts
 			(xy 217.17 118.11) (xy 214.63 118.11)
 		)
@@
 	(wire
 		(pts
+			(xy 170.18 227.33) (xy 170.18 238.76)
+		)
+		(stroke
+			(width 0)
+			(type default)
+		)
+	)
+	(wire
+		(pts
 			(xy 214.63 120.65) (xy 214.63 118.11)
 		)
@@
 	(wire
 		(pts
+			(xy 170.18 238.76) (xy 176.53 238.76)
+		)
+		(stroke
+			(width 0)
+			(type default)
+		)
+	)
+	(wire
+		(pts
 			(xy 204.47 119.38) (xy 204.47 113.03)
 		)
@@
 	(wire
 		(pts
+			(xy 154.94 236.22) (xy 154.94 241.3)
+		)
+		(stroke
+			(width 0)
+			(type default)
+		)
+	)
+	(wire
+		(pts
 			(xy 40.64 224.79) (xy 40.64 229.87)
 		)
@@
 	)
 	(label "VBUS"
-		(at 139.7 78.74 0)
+		(at 139.7 71.12 0)
 		(fields_autoplaced yes)
 		(effects
@@
 	)
 	(label "CC1"
-		(at 156.21 78.74 180)
+		(at 156.21 71.12 180)
 		(fields_autoplaced yes)
 		(effects
@@
 	)
 	(label "CC2"
-		(at 173.99 78.74 0)
+		(at 173.99 71.12 0)
 		(fields_autoplaced yes)
 		(effects
@@
 	(symbol
 		(lib_id "Device:D_TVS_Dual_AAC")
-		(at 165.1 78.74 0)
+		(at 165.1 71.12 0)
 		(unit 1)
 		(exclude_from_sim no)
@@
 		(fields_autoplaced yes)
 		(property "Reference" "D2"
-			(at 165.1 73.66 0)
+			(at 165.1 66.04 0)
 			(effects
 				(font
@@
 		)
 		(property "Value" "D_TVS_Dual_AAC"
-			(at 165.1 76.2 0)
+			(at 165.1 68.58 0)
 			(effects
 				(font
@@
 		)
 		(property "Footprint" "Package_TO_SOT_SMD:SOT-23"
-			(at 161.29 78.74 0)
+			(at 161.29 71.12 0)
 			(effects
 				(font
@@
 		)
 		(property "Datasheet" "~"
-			(at 161.29 78.74 0)
+			(at 161.29 71.12 0)
 			(effects
 				(font
@@
 		)
 		(property "Description" "Bidirectional dual transient-voltage-suppression diode, center on pin 3"
-			(at 165.1 78.74 0)
+			(at 165.1 71.12 0)
 			(effects
 				(font
@@
 		)
 		(property "LCSC" "C32677"
-			(at 165.1 78.74 0)
+			(at 165.1 71.12 0)
 			(effects
 				(font
@@
 	)
 	(symbol
+		(lib_id "power:GND")
+		(at 154.94 241.3 0)
+		(unit 1)
+		(exclude_from_sim no)
+		(in_bom yes)
+		(on_board yes)
+		(dnp no)
+		(fields_autoplaced yes)
+		(property "Reference" "#PWR026"
+			(at 154.94 247.65 0)
+			(effects
+				(font
+					(size 1.27 1.27)
+				)
+				(hide yes)
+			)
+		)
+		(property "Value" "GND"
+			(at 154.94 246.38 0)
+			(effects
+				(font
+					(size 1.27 1.27)
+				)
+			)
+		)
+		(property "Footprint" ""
+			(at 154.94 241.3 0)
+			(effects
+				(font
+					(size 1.27 1.27)
+				)
+				(hide yes)
+			)
+		)
+		(property "Datasheet" ""
+			(at 154.94 241.3 0)
+			(effects
+				(font
+					(size 1.27 1.27)
+				)
+				(hide yes)
+			)
+		)
+		(property "Description" "Power symbol creates a global label with name \"GND\" , ground"
+			(at 154.94 241.3 0)
+			(effects
+				(font
+					(size 1.27 1.27)
+				)
+				(hide yes)
+			)
+		)
+		(pin "1"
+		)
+		(instances
+			(project "Landing-Light"
+				(path "/f89d3217-1b1a-43a4-8c74-9ff6f0eaa6ee"
+					(reference "#PWR026")
+					(unit 1)
+				)
+			)
+		)
+	)
+	(symbol
 		(lib_id "Device:FerriteBead_Small")
 		(at 125.73 46.99 90)
@@
 	(symbol
 		(lib_id "power:GND")
-		(at 165.1 86.36 0)
+		(at 165.1 78.74 0)
 		(unit 1)
 		(exclude_from_sim no)
@@
 		(fields_autoplaced yes)
 		(property "Reference" "#PWR018"
-			(at 165.1 92.71 0)
+			(at 165.1 85.09 0)
 			(effects
 				(font
@@
 		)
 		(property "Value" "GND"
-			(at 165.1 91.44 0)
+			(at 165.1 83.82 0)
 			(effects
 				(font
@@
 		)
 		(property "Footprint" ""
-			(at 165.1 86.36 0)
+			(at 165.1 78.74 0)
 			(effects
 				(font
@@
 		)
 		(property "Datasheet" ""
-			(at 165.1 86.36 0)
+			(at 165.1 78.74 0)
 			(effects
 				(font
@@
 		)
 		(property "Description" ""
-			(at 165.1 86.36 0)
+			(at 165.1 78.74 0)
 			(effects
 				(font
@@
 	(symbol
 		(lib_id "power:GND")
-		(at 130.81 86.36 0)
+		(at 130.81 78.74 0)
 		(unit 1)
 		(exclude_from_sim no)
@@
 		(fields_autoplaced yes)
 		(property "Reference" "#PWR014"
-			(at 130.81 92.71 0)
+			(at 130.81 85.09 0)
 			(effects
 				(font
@@
 		)
 		(property "Value" "GND"
-			(at 130.81 91.44 0)
+			(at 130.81 83.82 0)
 			(effects
 				(font
@@
 		)
 		(property "Footprint" ""
-			(at 130.81 86.36 0)
+			(at 130.81 78.74 0)
 			(effects
 				(font
@@
 		)
 		(property "Datasheet" ""
-			(at 130.81 86.36 0)
+			(at 130.81 78.74 0)
 			(effects
 				(font
@@
 		)
 		(property "Description" ""
-			(at 130.81 86.36 0)
+			(at 130.81 78.74 0)
 			(effects
 				(font
@@
 	(symbol
 		(lib_id "Device:D_TVS_Dual_AAC")
-		(at 130.81 78.74 0)
+		(at 130.81 71.12 0)
 		(unit 1)
 		(exclude_from_sim no)
@@
 		(fields_autoplaced yes)
 		(property "Reference" "D4"
-			(at 130.81 73.66 0)
+			(at 130.81 66.04 0)
 			(effects
 				(font
@@
 		)
 		(property "Value" "D_TVS_Dual_AAC"
-			(at 130.81 76.2 0)
+			(at 130.81 68.58 0)
 			(effects
 				(font
@@
 		)
 		(property "Footprint" "Package_TO_SOT_SMD:SOT-23"
-			(at 127 78.74 0)
+			(at 127 71.12 0)
 			(effects
 				(font
@@
 		)
 		(property "Datasheet" "~"
-			(at 127 78.74 0)
+			(at 127 71.12 0)
 			(effects
 				(font
@@
 		)
 		(property "Description" "Bidirectional dual transient-voltage-suppression diode, center on pin 3"
-			(at 130.81 78.74 0)
+			(at 130.81 71.12 0)
 			(effects
 				(font
@@
 		)
 		(property "LCSC" "C32677"
-			(at 130.81 78.74 0)
+			(at 130.81 71.12 0)
 			(effects
 				(font

Commit message: Routing complete
Parts:
- removed D1: Schottky, Diode_SMD:D_SMA, symbol Device:D_Schottky
- removed J3: Conn_01x04, Connector_PinHeader_2.54mm:PinHeader_1x04_P2.54mm_Vertical, symbol Connector_Generic:Conn_01x04
- removed JP1, JP4: Jumper_2_Open, Jumper:SolderJumper-2_P1.3mm_Open_Pad1.0x1.5mm, symbol Jumper:Jumper_2_Open
- removed Q1: PMOS, Package_TO_SOT_SMD:SOT-23, symbol Simulation_SPICE:PMOS
- removed R14: 100k, Resistor_SMD:R_0603_1608Metric, symbol Device:R_US
- removed R21: R_US, Resistor_SMD:R_0603_1608Metric, symbol Device:R_US
- added C3: 47uF, Capacitor_SMD:C_0603_1608Metric, symbol Device:C_Small
- added JP5, JP6: Jumper_2_Open, Jumper:SolderJumper-2_P1.3mm_Open_RoundedPad1.0x1.5mm, symbol Jumper:Jumper_2_Open
- added Q3: NMOS, Package_TO_SOT_SMD:SOT-23-3, symbol Simulation_SPICE:NMOS
- added Q4: PMOS, Package_TO_SOT_SMD:SOT-23, symbol Simulation_SPICE:PMOS
- added R10: 1M, Resistor_SMD:R_0603_1608Metric, symbol Device:R_US
- added R11: 180k, Resistor_SMD:R_0603_1608Metric, symbol Device:R_US
- added TP1: VCC, TestPoint:TestPoint_Pad_D1.0mm, symbol Connector:TestPoint
- added TP4: -BATT, TestPoint:TestPoint_Pad_D1.0mm, symbol Connector:TestPoint
- added TP7: VIN, TestPoint:TestPoint_Pad_D1.0mm, symbol Connector:TestPoint
- JP2, JP3: footprint Jumper:SolderJumper-2_P1.3mm_Open_Pad1.0x1.5mm -> Jumper:SolderJumper-2_P1.3mm_Open_RoundedPad1.0x1.5mm
- R19: value R_US -> 0R; LCSC (none) -> C17168
- R20: value R_US -> 100k; LCSC (none) -> C25803
- TP2: value VCC -> 5V
- TP3: value VBUS -> GND
Connections:
- net +3V3: now also C3.1, R10.1; no longer R20.1
- net +BATT: now also C12.1, L2.1, U3.5 (VIN), U3.6 (EN), U3.7 (UVLO), U3.8 (PS), TP1.1
- net -BATT: now also JP5.1 (A), Q3.3 (S), TP4.1; no longer C1.1, C10.2, C11.2, C12.2, C13.2, C2.1, C8.2, C9.1, D2.3 (common), D3.3 (common), D4.3 (common), J1.1 (Pin_1), J2.A1 (GND1), J2.A12 (GND2), J2.B1 (GND3), J2.B12 (GND4), J2.S1 (SHIELD), J2.S2 (SHIELD), J2.S3 (SHIELD), J2.S4 (SHIELD), R12.1, R15.2, R18.2, R19.2, R2.2, R3.2, R4.2, R5.2, SW3.1 (A), U1.4 (GND), U1.9 (EXP), U3.11 (PAD), U3.4 (PGND), U3.9 (GND)
- net VAUX: now reaches C13.1, U3.1 (VAUX)
- net VAUX: now also Q3.2 (G)
- net at U3.10 (FB): now also R10.2, R11.1; no longer R20.2
- net VBUS renamed +5V
- net +5V: now also R20.1, TP2.1, Q4.1 (G); no longer D4.2 (A2), TP3.1
- removed net VCC: C12.1, L2.1, TP2.1, U3.5 (VIN), U3.6 (EN), U3.7 (UVLO), U3.8 (PS)
- net VSS renamed VIN
- net VIN: now also D4.2 (A2), TP7.1
- new net: JP6.1 (A), Q4.3 (D), SW3.1 (A)
- new net GND: C1.1, C10.2, C11.2, C12.2, C13.2, C2.1, C3.2, C8.2, C9.1, D2.3 (common), D3.3 (common), D4.3 (common), J1.1 (Pin_1), J2.A1 (GND1), J2.A12 (GND2), J2.B1 (GND3), J2.B12 (GND4), J2.S1 (SHIELD), J2.S2 (SHIELD), J2.S3 (SHIELD), J2.S4 (SHIELD), JP5.2 (B), JP6.2 (B), Q3.1 (D), Q4.2 (S), R11.2, R12.1, R15.2, R18.2, R19.2, R2.2, R20.2, R3.2, R4.2, R5.2, TP3.1, U1.4 (GND), U1.9 (EXP), U3.11 (PAD), U3.4 (PGND), U3.9 (GND)
Other:
- note added: "2mA here"
- note added: "9-10mA here"
- note removed: "Battery reverse polarity protection"
- moved on the sheet: C1, C10, C11, C12, C13, C2, C8, C9, D2, D3, D4, D6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

Commit message: Layout labelling
Other:
- note added: "3.3v Regulator"
- note added: "Battery Charger"
- note added: "Battery and reverse polarity protection"
- note added: "Charging LED"
- note added: "RGB LED"
Changed lines of the file:
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@@
+		)
+	)
+	(text "Battery \nand reverse polarity protection"
+		(exclude_from_sim no)
+		(at 131.318 34.29 0)
+		(effects
+			(font
+				(size 3 3)
+				(bold yes)
+				(color 0 0 255 1)
+			)
+			(justify left bottom)
+		)
+	)
+	(text "RGB LED"
+		(exclude_from_sim no)
+		(at 359.156 23.622 0)
+		(effects
+			(font
+				(size 3 3)
+				(bold yes)
+				(color 0 0 255 1)
+			)
+			(justify left bottom)
 		)
 	)
@@
 		)
 	)
+	(text "3.3v Regulator"
+		(exclude_from_sim no)
+		(at 211.074 31.496 0)
+		(effects
+			(font
+				(size 3 3)
+				(bold yes)
+				(color 0 0 255 1)
+			)
+			(justify left bottom)
+		)
+	)
+	(text "Battery Charger"
+		(exclude_from_sim no)
+		(at 17.526 27.94 0)
+		(effects
+			(font
+				(size 3 3)
+				(bold yes)
+				(color 0 0 255 1)
+			)
+			(justify left bottom)
+		)
+	)
+	(text "Charging LED"
+		(exclude_from_sim no)
+		(at 297.18 28.702 0)
+		(effects
+			(font
+				(size 3 3)
+				(bold yes)
+				(color 0 0 255 1)
+			)
+			(justify left bottom)
+		)
+	)
