File: hardware/pcb/Landing-Light/Landing-Light.kicad_sch (KiCad schematic)
At the start: 53 parts, among them J1 Conn_01x04, J2 2012670005, Q2 NMOS, Q3 NMOS, Q4 PMOS, SW1 SW_SPDT, SW2 SW_SP3T, U1 BQ25172DSGR, U3 TPS61200DRC

Commit message: Complete redesign - starting point
Parts:
- removed D2, D3, D4: D_TVS_Dual_AAC, Package_TO_SOT_SMD:SOT-23, symbol Device:D_TVS_Dual_AAC
- removed J2: 2012670005, Landing-Light:MOLEX_2012670005, symbol ESP32_Dev_Board-eagle-import:2012670005
- removed R1, R8, R9: 75R, Resistor_SMD:R_0402_1005Metric, symbol Device:R_US
- added J3: USB_C_Receptacle_USB2.0_16P, Connector_USB:USB_C_Receptacle_G-Switch_GT-USB-7010ASV, symbol Connector:USB_C_Receptacle_USB2.0_16P
- added R8: TC33X-2-501E, Potentiometer_SMD:Potentiometer_Bourns_TC33X_Vertical, symbol Device:R_Variable
- added U2: SRV05-4, Package_TO_SOT_SMD:SOT-363_SC-70-6, symbol Power_Protection:SRV05-4
Connections:
- net CC1: now also R12.1, J3.A5 (CC1), U2.4 (IO3); no longer R12.2
- net CC2: now also J3.B5 (CC2), U2.6 (IO4)
- net CHARGE_STATUS: now also U2.1 (IO1)
- net DATA2: now also U2.3 (IO2)
- net GND: now also R12.2, J3.A1 (GND), J3.A12 (GND), J3.B1 (GND), J3.B12 (GND), J3.S1 (SHIELD), U2.2 (VN); no longer R12.1
- net VIN: now also J3.A4 (VBUS), J3.A9 (VBUS), J3.B4 (VBUS), J3.B9 (VBUS), U2.5 (VP)
- net B: now reaches SW2.1
- net B: now also D7.4 (BA)
- net R_R: now reaches SW2.4
- net R_R: now also R13.1
- net TS: now reaches R2.1, U1.3 (TS)
- net VCC_SW: now reaches C12.1, JP4.1 (A), L2.1, R3.1, SW1.1 (A), U3.5 (VIN), U3.6 (EN), U3.8 (PS)
- net L: now reaches L2.2, U3.3 (L)
- net ISET: now reaches R6.1, U1.2 (ISET)
- net TMR: now reaches R7.1, U1.6 (TMR)
- net VSET: now reaches R5.1, U1.7 (VSET)
- net UVLO: now reaches JP4.2 (B), R3.2, R4.1, U3.7 (UVLO)
- net G: now reaches SW2.2
- net G: now also D7.3 (GA)
- net Anode_R: now reaches Q2.1 (D), Q4.3 (D)
- net Anode_R: now also R8.2; no longer D7.2 (K)
- net R: now reaches D7.1 (RA), R13.2
- net FB: now reaches R10.2, R11.1, U3.10 (FB)
- new net Anode: D7.2 (K), R8.1
- no-connect marks 16 -> 7
Other:
- note removed: "10%"
- moved on the sheet: D7, R12, R13, R15, SW2
