File: hardware/pcb/Landing-Light/Landing-Light.kicad_pcb (KiCad board)
At the start: 2 copper layers, 70 x 20 mm, 56 parts, among them J1 Conn_01x04, J2 2012670005, Q2 NMOS, Q3 NMOS, Q4 PMOS, SW2 SW_SP3T, SW3 SW_SPDT, U1 BQ25172DSGR, U3 TPS61200DRC

Commit message: Final layout checks
Parts:
- removed R17: 100R, Resistor_SMD:R_0402_1005Metric
- added JP4: Jumper_2_Open, Jumper:SolderJumper-2_P1.3mm_Open_RoundedPad1.0x1.5mm, B.Cu at (170.1, 89.7)
- Q2, Q3: footprint Package_TO_SOT_SMD:SOT-23-3 -> Landing-Light:SOT-23-3-JLCPCB
- R1, R13: value 330R -> 75R
- R19: value 0R -> 220R
- R8, R9: value 100R -> 75R
- moved R4 4.39 mm to (173.7, 88.9)
- moved R3 4.25 mm to (171.2, 88.9)
- moved TP1 3.14 mm to (175.0, 89.6)
- moved R9 2.01 mm to (128.2, 90.0)
- moved R1 0.94 mm to (131.2, 88.5)
- moved R8 0.74 mm to (131.2, 90.0), turned to 180 degrees
- moved TP4 0.25 mm to (126.5, 91.8)
- moved Q2 0.21 mm to (149.1, 94.3), turned to 90 degrees
- moved Q3 0.09 mm to (131.5, 94.8), turned to 0 degrees
- turned JP5 to 90 degrees
- turned R18 to 90 degrees
Connections:
- R3 pad 1: unconnected-(R3-Pad1) -> +BATT
- R3 pad 2: unconnected-(R3-Pad2) -> Net-(JP4-B)
- R4 pad 1: unconnected-(R4-Pad1) -> Net-(JP4-B)
- R4 pad 2: unconnected-(R4-Pad2) -> GND
- R9 pad 2: Net-(R17-Pad1) -> Net-(D7-BA)
- U3 pad 7: +BATT -> Net-(JP4-B)
Routing:
- net +BATT: track 12.1 -> 25.3 mm, vias 1 -> 2
- net Net-(JP4-B): track 0.00 -> 8.61 mm, vias 0 -> 2
- net +3V3: track 31.0 -> 34.5 mm
- net GND: track 46.4 -> 43.9 mm, vias 30 -> 33
- net Net-(R1-Pad2): track 0.00 -> 1.94 mm
- net Net-(R9-Pad1): track 13.5 -> 15.3 mm
- net -BATT: track 10.7 -> 12.1 mm
- net Net-(R1-Pad1): track 6.48 -> 5.45 mm
- net Net-(Q2-S): track 2.76 -> 1.78 mm
- net Net-(D7-GA): track 9.76 -> 8.84 mm
- net VAUX: track 40.4 -> 39.5 mm
- net Net-(JP3-A): track 1.77 -> 2.56 mm
- net Net-(D7-K): track 31.2 -> 31.8 mm
Other:
- board text added: "UVLO"
