File: hardware/pcb/Landing-Light/Landing-Light.kicad_pcb (KiCad board)
At the start: 2 copper layers, 62.8 x 21 mm, 51 parts, among them J1 Conn_01x04, J3 USB_C_Receptacle_USB2.0_16P, Q2 NMOS, Q3 NMOS, Q4 PMOS, SW1 SW_SPDT, SW2 SW_SP3T, U1 BQ25172DSGR, U2 SRV05-4, U3 TPS61200DRC

Commit message: Clean ground plane
Parts:
- added R14: 0R, Resistor_SMD:R_0402_1005Metric, F.Cu at (126.8, 87.8)
- added R17: 0R, Resistor_SMD:R_0402_1005Metric, F.Cu at (126.8, 90.0)
- moved TP1 3.69 mm to (170.8, 92.0)
Connections:
- SW2 pad 1: /B -> Net-(R17-Pad1)
- SW2 pad 2: /G -> Net-(R14-Pad1)
- U2 pad 3: DATA2 -> unconnected-(U2-IO2-Pad3)
Routing:
- net /B: track 22.9 -> 5.94 mm, vias 0 -> 1
- net Net-(R17-Pad1): track 0.00 -> 16.5 mm
- net /G: track 23.3 -> 10.3 mm
- net Net-(R14-Pad1): track 0.00 -> 11.9 mm
- net DATA2: track 2.66 -> 0.00 mm
- net /Anode: track 11.5 -> 10.5 mm
- net /VCC_SW: track 27.4 -> 28.1 mm
- net GND: track 42.0 -> 42.2 mm, vias 42 -> 45

Commit message: Finalise BOM
Parts:
- R12, R15, R19: footprint Resistor_SMD:R_0603_1608Metric -> Resistor_SMD:R_0402_1005Metric
- R16: value 330R -> 1.5k
- R18, R20: value 100k -> 150k; footprint Resistor_SMD:R_0603_1608Metric -> Resistor_SMD:R_0402_1005Metric
- moved TP5 1.30 mm to (166.3, 92.0)
- moved R12 1.09 mm to (126.7, 100.4), turned to 0 degrees
- moved J1 0.85 mm to (179.2, 101.6)
- moved TP7 0.80 mm to (179.2, 92.1)
- moved R15 0.73 mm to (126.7, 103.3), turned to 0 degrees
- moved H1 0.71 mm to (179.5, 105.5)
- moved H2 0.71 mm to (179.5, 89.5)
- moved J3 0.55 mm to (120.3, 101.6)
- moved R19 0.43 mm to (141.1, 95.2)
- moved R18 0.41 mm to (136.5, 95.2)
- moved R20 0.35 mm to (146.2, 95.2)
- moved R8 0.20 mm to (132.9, 94.4)
Routing:
- net CHARGE_STATUS: track 26.8 -> 24.1 mm
- net GND: track 42.2 -> 41.3 mm, vias 45 -> 48
- net /CC1: track 59.1 -> 58.5 mm
- net VIN: track 110.0 -> 110.4 mm, vias 2 -> 3
Other:
- board size 62.8 x 21 mm -> 63.5 x 21 mm
- board text added: "NC"

Commit message: v1.1 production
Routing:
- net CHARGE_STATUS: track 24.1 -> 27.6 mm
- net GND: track 41.3 -> 39.7 mm, vias 48 -> 43
- net VIN: track 110.4 -> 111.6 mm
Changed lines of the file:
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@@
 		(sheetname "/")
 		(sheetfile "Landing-Light.kicad_sch")
-		(attr smd)
+		(attr smd exclude_from_bom dnp)
 		(fp_line
 			(start -0.140581 -0.51)
@@
 	(gr_poly
 		(pts
-			(xy 156.91 95.86) (xy 156.47 94.55) (xy 156.36 94.55) (xy 155.92 95.86) (xy 156.15 95.86) (xy 156.41 94.99)
-			(xy 156.68 95.86)
+			(xy 157.16 96.11) (xy 156.72 94.8) (xy 156.61 94.8) (xy 156.17 96.11) (xy 156.4 96.11) (xy 156.66 95.24)
+			(xy 156.93 96.11)
 		)
 		(stroke
@@
 		(layer "Edge.Cuts")
 	)
+	(gr_text "Landing Light\nv1.1"
+		(at 157.75 94.25 0)
+		(layer "F.SilkS")
+		(effects
+			(font
+				(size 0.66 0.66)
+				(thickness 0.1)
+			)
+			(justify bottom)
+		)
+	)
 	(gr_text "TT"
-		(at 158 95.25 -0)
+		(at 158.25 95.5 -0)
 		(layer "F.SilkS")
 		(effects
@@
 			(polygon
 				(pts
-					(xy 157.350711 95.8725) (xy 157.350711 94.765438) (xy 156.999459 94.765438) (xy 156.999459 94.565312)
-					(xy 157.9488 94.565312) (xy 157.9488 94.765438) (xy 157.579047 94.765438) (xy 157.579047 95.8725)
+					(xy 157.601535 96.1225) (xy 157.601535 95.014614) (xy 157.249001 95.014614) (xy 157.249001 94.815312)
+					(xy 158.199625 94.815312) (xy 158.199625 95.014614) (xy 157.828223 95.014614) (xy 157.828223 96.1225)
 				)
 			)
 			(polygon
 				(pts
-					(xy 158.399978 95.8725) (xy 158.399978 94.765438) (xy 158.048726 94.765438) (xy 158.048726 94.565312)
-					(xy 158.998068 94.565312) (xy 158.998068 94.765438) (xy 158.628314 94.765438) (xy 158.628314 95.8725)
+					(xy 158.650802 96.1225) (xy 158.650802 95.014614) (xy 158.298268 95.014614) (xy 158.298268 94.815312)
+					(xy 159.248892 94.815312) (xy 159.248892 95.014614) (xy 158.87749 95.014614) (xy 158.87749 96.1225)
 				)
 			)
@@
 		)
 	)
-	(gr_text "Landing Light v1.1"
-		(at 157.5 95.75 0)
-		(layer "B.SilkS")
-		(effects
-			(font
-				(size 1 1)
-				(thickness 0.1)
-			)
-			(justify bottom mirror)
-		)
-	)
 	(gr_text "GND"
 		(at 180.2 101.5 270)
@@
 	)
 	(segment
-		(start 127.2 103.3)
-		(end 127.75 102.75)
-		(width 0.3)
-		(layer "F.Cu")
-		(net 3)
-	)
-	(segment
 		(start 147.595998 90.024)
 		(end 147.671998 90.1)
@@
 	)
 	(segment
-		(start 127.75 102.75)
-		(end 127.75 102.05)
-		(width 0.3)
-		(layer "F.Cu")
-		(net 3)
-	)
-	(segment
 		(start 164.0115 93.261499)
 		(end 165.0615 93.261499)
@@
 	)
 	(segment
-		(start 127.75 102.05)
-		(end 127.7 102)
-		(width 0.3)
-		(layer "F.Cu")
-		(net 3)
-	)
-	(segment
 		(start 171.31538 93.23462)
 		(end 171.27076 93.19)
@@
 	)
 	(via
-		(at 126.25 105.75)
-		(size 0.9)
-		(drill 0.4)
-		(layers "F.Cu" "B.Cu")
-		(free yes)
-		(net 3)
-	)
-	(via
 		(at 163.5 88.6)
 		(size 0.9)
@@
 	)
 	(via
-		(at 176.25 88.25)
-		(size 0.9)
-		(drill 0.4)
-		(layers "F.Cu" "B.Cu")
-		(free yes)
-		(net 3)
-	)
-	(via
-		(at 127.75 107.25)
-		(size 0.9)
-		(drill 0.4)
-		(layers "F.Cu" "B.Cu")
-		(free yes)
-		(net 3)
-	)
-	(via
 		(at 162.8 93.3)
 		(size 0.9)
@@
 	)
 	(via
-		(at 124.75 107.25)
-		(size 0.9)
-		(drill 0.4)
-		(layers "F.Cu" "B.Cu")
-		(free yes)
-		(net 3)
-	)
-	(via
 		(at 122.5 103.5)
 		(size 0.9)
@@
 	)
 	(via
-		(at 126.25 107.25)
-		(size 0.9)
-		(drill 0.4)
-		(layers "F.Cu" "B.Cu")
-		(free yes)
-		(net 3)
-	)
-	(via
 		(at 173.2 88.7)
 		(size 0.9)
@@
 	)
 	(via
-		(at 123.5 95)
+		(at 123.25 95)
 		(size 0.9)
 		(drill 0.4)
@@
 	)
 	(via
-		(at 127.75 105.75)
+		(at 178 98)
 		(size 0.9)
 		(drill 0.4)
@@
 	)
 	(via
-		(at 127.7 102)
-		(size 0.6)
-		(drill 0.3)
-		(layers "F.Cu" "B.Cu")
-		(free yes)
-		(net 3)
-	)
-	(via
 		(at 136.5 93.55)
 		(size 0.7)
@@
 		(net 3)
 	)
+	(via
+		(at 177 99)
+		(size 0.9)
+		(drill 0.4)
+		(layers "F.Cu" "B.Cu")
+		(free yes)
+		(net 3)
+	)
 	(segment
 		(start 169.520503 95.869497)
@@
 	)
 	(segment
+		(start 179.2 94.05)
+		(end 177.312499 95.937501)
+		(width 0.6)
+		(layer "F.Cu")
+		(net 6)
+	)
+	(segment
 		(start 179.2 93.959999)
-		(end 178.35 93.959999)
+		(end 179.2 94.05)
 		(width 0.6)
 		(layer "F.Cu")
@@
 	)
 	(segment
-		(start 179.359999 93.959999)
-		(end 180.8 95.4)
+		(start 176.475 97.5)
+		(end 176.475 96.212501)
+		(width 0.4)
+		(layer "F.Cu")
+		(net 6)
+	)
+	(segment
+		(start 181.4 102.6)
+		(end 180.5 103.5)
 		(width 0.3)
 		(layer "F.Cu")
@@
 	)
 	(segment
-		(start 178.35 93.959999)
-		(end 176.372498 95.937501)
-		(width 0.6)
+		(start 176.286418 103.5)
+		(end 175.365582 102.579164)
+		(width 0.3)
 		(layer "F.Cu")
 		(net 6)
 	)
 	(segment
-		(start 176.475 97.5)
-		(end 176.475 96.212501)
-		(width 0.4)
+		(start 181.4 96)
+		(end 181.4 102.6)
+		(width 0.3)
 		(layer "F.Cu")
 		(net 6)
 	)
 	(segment
-		(start 175.986418 103.2)
-		(end 175.365582 102.579164)
+		(start 179.2 93.959999)
+		(end 179.359999 93.959999)
 		(width 0.3)
 		(layer "F.Cu")
@@
 	)
 	(segment
+		(start 180.5 103.5)
+		(end 176.286418 103.5)
+		(width 0.3)
+		(layer "F.Cu")
+		(net 6)
+	)
+	(segment
 		(start 122.65 100.4)
 		(end 122.65 99.840298)
@@
 	)
 	(segment
-		(start 176.372498 95.937501)
-		(end 176.2 95.937501)
-		(width 0.6)
+		(start 175.365582 102.579164)
+		(end 175.365582 102.565582)
+		(width 0.3)
 		(layer "F.Cu")
 		(net 6)
@@
 	)
 	(segment
-		(start 180.8 95.4)
-		(end 180.8 102.5)
-		(width 0.3)
-		(layer "F.Cu")
-		(net 6)
-	)
-	(segment
-		(start 180.8 102.5)
-		(end 180.1 103.2)
-		(width 0.3)
-		(layer "F.Cu")
-		(net 6)
-	)
-	(segment
 		(start 122.65 99.840298)
 		(end 123.300298 99.19)
@@
 	)
 	(segment
-		(start 180.1 103.2)
-		(end 175.986418 103.2)
-		(width 0.3)
-		(layer "F.Cu")
-		(net 6)
-	)
-	(segment
 		(start 176.287496 97.5)
 		(end 176.224997 97.437501)
@@
 	)
 	(segment
-		(start 174.975 101.6)
-		(end 174.650001 101.6)
-		(width 0.3)
+		(start 177.312499 95.937501)
+		(end 176.2 95.937501)
+		(width 0.6)
 		(layer "F.Cu")
 		(net 6)
 	)
 	(segment
-		(start 175.365582 102.579164)
-		(end 175.365582 102.565582)
+		(start 174.975 101.6)
+		(end 174.650001 101.6)
 		(width 0.3)
 		(layer "F.Cu")
@@
 	)
 	(segment
-		(start 179.2 93.959999)
-		(end 179.359999 93.959999)
+		(start 179.359999 93.959999)
+		(end 181.4 96)
 		(width 0.3)
 		(layer "F.Cu")
@@
 	)
 	(segment
+		(start 180.8 98.1)
+		(end 180.8 102.3)
+		(width 0.25)
+		(layer "F.Cu")
+		(net 7)
+	)
+	(segment
 		(start 166.29 93.199999)
 		(end 166.29 92.5)
@@
 	)
 	(segment
-		(start 175.873999 100.526001)
-		(end 179.2 97.2)
-		(width 0.3)
+		(start 180.8 102.3)
+		(end 180.35 102.75)
+		(width 0.25)
 		(layer "F.Cu")
 		(net 7)
@@
 	)
 	(segment
-		(start 179.2 97.2)
-		(end 179.2 96.5)
-		(width 0.3)
-		(layer "F.Cu")
-		(net 7)
-	)
-	(segment
-		(start 176.55 102.25)
-		(end 176.225001 102.25)
-		(width 0.3)
+		(start 166.3615 93.271499)
+		(end 166.29 93.199999)
+		(width 0.2)
 		(layer "F.Cu")
 		(net 7)
 	)
 	(segment
-		(start 166.3615 93.271499)
-		(end 166.29 93.199999)
-		(width 0.2)
+		(start 179.2 96.5)
+		(end 180.8 98.1)
+		(width 0.25)
 		(layer "F.Cu")
 		(net 7)
 	)
 	(segment
-		(start 176.225001 102.25)
-		(end 175.873999 101.898998)
-		(width 0.3)
+		(start 180.35 102.75)
+		(end 177.05 102.75)
+		(width 0.25)
 		(layer "F.Cu")
 		(net 7)
 	)
 	(segment
-		(start 175.873999 101.898998)
-		(end 175.873999 100.526001)
-		(width 0.3)
+		(start 177.05 102.75)
+		(end 176.55 102.25)
+		(width 0.25)
 		(layer "F.Cu")
 		(net 7)

Commit message: v1.2 Production
Parts:
- removed C11, C12: 10uF, Capacitor_SMD:C_0603_1608Metric
- removed D7: LED_RKGB, LED_THT:LED_D5.0mm-4_RGB
- removed J1: Conn_01x04, MHCI:399-10-104-10-008000
- removed Q2: NMOS, Landing-Light:SOT-23-3-JLCPCB
- removed R14, R17: 0R, Resistor_SMD:R_0402_1005Metric
- removed R16: 1.5k, Resistor_SMD:R_0402_1005Metric
- removed R18: 150k, Resistor_SMD:R_0402_1005Metric
- removed R19: 220R, Resistor_SMD:R_0402_1005Metric
- removed TP5: STATUS, TestPoint:TestPoint_Pad_D1.0mm
- added C4: 4.7uF, Capacitor_SMD:C_0805_2012Metric, F.Cu at (146.7, 92.1)
- added D1: LED_GBAR, LED_THT:LED_D5.0mm-4_RGB_Wide_Pins, F.Cu at (122.5, 88.2)
- added J2: Conn_01x02, 399-10-102-10-008000:HDRRA2W46P0X254_1X2_508X279X254P, F.Cu at (179.2, 94.0)
- added JP1: PS Bridge, Jumper:SolderJumper-3_P1.3mm_Bridged2Bar12_RoundedPad1.0x1.5mm, F.Cu at (158.2, 93.1)
- added JP2: CHG_LED, Jumper:SolderJumper-3_P1.3mm_Bridged2Bar12_RoundedPad1.0x1.5mm, F.Cu at (142.9, 91.7)
- added JP3: 5V_PMOS, Landing-Light:SolderJumper-2_P1.3mm_Open_RoundedPad0.5x0.75mm, F.Cu at (138.6, 93.8)
- added JP5: SolderJumper_2_Open, Landing-Light:SolderJumper-2_P1.3mm_Open_RoundedPad0.5x0.75mm, F.Cu at (131.3, 91.5)
- added Q1: NMOS, Landing-Light:SOT-23-3-JLCPCB, F.Cu at (170.2, 89.4)
- added R1: 5.6k, Resistor_SMD:R_0402_1005Metric, F.Cu at (132.9, 93.2)
- C3: value 47uF -> 4.7uF; footprint Capacitor_SMD:C_0603_1608Metric -> Capacitor_SMD:C_0805_2012Metric
- C8: value 10uF -> 4.7uF; footprint Capacitor_SMD:C_0603_1608Metric -> Capacitor_SMD:C_0805_2012Metric
- JP4: value Jumper_2_Open -> 5V_LED_ON; footprint Jumper:SolderJumper-2_P1.3mm_Open_RoundedPad1.0x1.5mm -> Landing-Light:SolderJumper-2_P1.3mm_Bridged_RoundedPad0.5x0.75mm; moved to F.Cu
- R13: value 75R -> 150k
- R3: value 510k -> 470k
- R4: value 200k -> 150k
- R8: value TC33X-2-501E -> 1.5k; footprint Potentiometer_SMD:Potentiometer_Bourns_TC33X_Vertical -> Resistor_SMD:R_0402_1005Metric
- SW1: value SW_SPDT -> ON_OFF
- SW2: value SW_SP3T -> LED_COL
- TP1, TP2, TP3, TP4, TP6, TP7: moved to F.Cu
- moved TP3 50.9 mm to (176.0, 98.0), turned to 0 degrees
- moved C10 49.1 mm to (125.7, 97.0), turned to -90 degrees
- moved C9 49.1 mm to (125.7, 98.9), turned to -90 degrees
- moved U2 49.0 mm to (126.7, 105.3), turned to -90 degrees
- moved FB1 49.0 mm to (127.3, 98.1)
- moved C8 48.6 mm to (127.3, 101.7), turned to -90 degrees
- moved TP4 44.5 mm to (176.0, 94.0), turned to 0 degrees
- moved R13 41.3 mm to (167.9, 92.4), turned to -90 degrees
- moved TP2 35.8 mm to (140.5, 94.9)
- moved D6 26.4 mm to (143.3, 94.0), turned to 180 degrees
- moved JP4 16.7 mm to (169.5, 93.0), turned to 90 degrees
- moved R20 13.3 mm to (132.9, 95.1)
- moved R8 11.0 mm to (143.9, 95.5)
- moved C3 9.19 mm to (154.1, 90.5)
- moved Q4 8.45 mm to (135.4, 94.3), turned to 180 degrees
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Connections:
- C1 pad 1: GND -> -BATT
- C10 pad 2: GND -> -BATT
- C2 pad 1: GND -> -BATT
- C3 pad 1: +3V3 -> /VCC_SW
- C8 pad 2: GND -> -BATT
- C9 pad 1: GND -> -BATT
- J3 pad A1: GND -> -BATT
- J3 pad A12: GND -> -BATT
- J3 pad B1: GND -> -BATT
- J3 pad B12: GND -> -BATT
- J3 pad S1: GND -> -BATT
- JP4 pad 1: /VCC_SW -> +5V
- JP4 pad 2: /UVLO -> Net-(JP4-B)
- Q4 pad 2: GND -> /Switch_Cathode
- Q4 pad 3: /Anode_R -> Net-(JP3-A)
- R12 pad 2: GND -> -BATT
- R13 pad 1: /R_R -> Net-(JP4-B)
- R13 pad 2: /R -> -BATT
- R15 pad 2: GND -> -BATT
- R2 pad 2: GND -> -BATT
- R5 pad 2: GND -> -BATT
- R6 pad 2: GND -> -BATT
- R7 pad 2: GND -> -BATT
- R8 pad 1: /Anode -> Net-(JP2-C)
- R8 pad 2: /Anode_R -> CHARGE_STATUS
- SW2 pad 1: Net-(R17-Pad1) -> /R
- SW2 pad 2: Net-(R14-Pad1) -> /G
- SW2 pad 3: +3V3 -> /Switch_Cathode
- SW2 pad 4: /R_R -> /B
- U1 pad 4: GND -> -BATT
- U1 pad 9: GND -> -BATT
- U2 pad 1: CHARGE_STATUS -> unconnected-(U2-IO1-Pad1)
- U2 pad 2: GND -> -BATT
- U2 pad 4: /CC1 -> /CC2
- U2 pad 6: /CC2 -> /CC1
- U3 pad 8: /VCC_SW -> /PS
Routing:
- net /CC2: track 67.2 -> 6.73 mm
- net /CC1: track 58.5 -> 10.2 mm
- net GND: track 39.7 -> 8.87 mm, vias 43 -> 30
- net -BATT: track 5.46 -> 35.2 mm, vias 0 -> 15
- net /R: track 3.98 -> 23.8 mm, vias 0 -> 2
- net VIN: track 111.6 -> 93.9 mm, vias 3 -> 1
- net Net-(R17-Pad1): track 16.5 -> 0.00 mm
- net +3V3: track 22.5 -> 37.0 mm, vias 1 -> 2
- net /PS: track 0.00 -> 13.3 mm, vias 0 -> 2
- net Net-(R14-Pad1): track 11.9 -> 0.00 mm
- net /Anode_R: track 10.6 -> 0.00 mm
- net /Anode: track 10.5 -> 0.00 mm
- net CHARGE_STATUS: track 27.6 -> 20.4 mm, vias 1 -> 2
- net Net-(JP4-B): track 0.00 -> 6.80 mm
- net /R_R: track 6.74 -> 0.00 mm
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- added copper zone on B.Cu, net -BATT
- added copper zone on F.Cu, net -BATT
Other:
- board text added: "+"
- board text added: "B+"
- board text added: "B-"
- board text added: "CHG LED"
- board text added: "GND NMOS"
- board text added: "LED PMOS"
- board text added: "Landing Light v1.2"
- board text added: "PS"
- board text added: "VREG NMOS"
- board text removed: "-BATT"
- board text removed: "BATT+"
- board text removed: "CHRG"
- board text removed: "Landing Light v1.1"
- board text removed: "NC"
- board text removed: "STAT"
- board text removed: "UVLO"
